Commit message: no idea

File: jackal_description/urdf/jackal2.urdf.xacro (robot description, xacro)
@@ -81,5 +81,5 @@
   <link name="base_link"></link>
   <joint name="base_link_joint" type="fixed">
-    <origin xyz="0 0 0" rpy="0 0 0" />
+    <origin xyz="-10 0 0" rpy="0 0 0" />
     <parent link="base_link"/>
     <child link="chassis_link" />

Commit message: fix urdf

File: jackal_description/urdf/jackal2.urdf.xacro (robot description, xacro)
@@ -81,5 +81,5 @@
   <link name="base_link"></link>
   <joint name="base_link_joint" type="fixed">
-    <origin xyz="-10 0 0" rpy="0 0 0" />
+    <origin xyz="0 0 0" rpy="0 0 0" />
     <parent link="base_link"/>
     <child link="chassis_link" />
